Commit message: feat: import velodyne driver package and update roboteq driver configuration

File: src/sirius/sirius_description/urdf/sirius3.urdf.xacro (robot description, xacro)
@@ -64,4 +64,11 @@
     <origin xyz="0.0 0.0 0.0" rpy="0 0 0"/>
   </joint>
+  <!-- Velodyne frame (Velodyne 3D LiDAR用) -->
+  <link name="${prefix}velodyne"/>
+  <joint name="${prefix}lidar_link_to_velodyne" type="fixed">
+    <parent link="${prefix}lidar_link"/>
+    <child link="${prefix}velodyne"/>
+    <origin xyz="0.0 0.0 0.0" rpy="0 0 0"/>
+  </joint>
   <!-- ======================================== -->
   <!-- IMU Link (ロボット中心)                   -->
